Commit message: Add inertial properties to vehicle model

File: src/senton_description/urdf/senton.urdf.xacro (robot description, xacro)
@@ -1,18 +1,5 @@
 <?xml version="1.0"?>
 <robot xmlns:xacro="http://www.ros.org/wiki/xacro" name="senton">
-    <!-- vehicle dimensions-->
-     <xacro:property name="vehicle_length" value="0.558"/>
-     <xacro:property name="vehicle_width" value="0.305"/>
-     <xacro:property name="vehicle_height" value="0.210"/>
-     <xacro:property name="vehicle_mass" value="3.55"/>
-     <xacro:property name= "wheelbase" value="0.327"/>
-    <!-- wheel dimensions-->
-     <xacro:property name="wheel_radius" value="0.052"/>
-     <xacro:property name="wheel_width" value="0.042"/>
-     <xacro:property name="track_width" value="0.263"/>
-    <xacro:property name="chassis_length" value="0.40"/>
-    <xacro:property name="chassis_width"  value="0.16"/>
-    <xacro:property name="chassis_height" value="0.09"/>
-    <xacro:property name="chassis_z"      value="0.03"/>
+   <xacro:include filename="$(find senton_description)/urdf/senton_properties.xacro"/>
     <link name="base_footprint"/>
         <joint name="base_footprint_joint" type="fixed">
@@ -31,4 +18,11 @@
         </material>
     </visual>
+    <xacro:box_inertia
+        m="${chassis_mass}"
+        x="${chassis_length}"
+        y="${chassis_width}"
+        z="${chassis_height}"
+        o_xyz="0 0 ${chassis_z}"
+        o_rpy="0 0 0"/>
 </link>
     <!-- Wheel macro -->
@@ -52,4 +46,10 @@
             </material>
         </visual>
+        <xacro:cylinder_inertia
+            m="${wheel_mass}"
+            r="${wheel_radius}"
+            l="${wheel_width}"
+            o_xyz="0 0 0"
+            o_rpy="${pi/2} 0 0"/>
     </link>
 </xacro:macro>

Commit message: Add Gazebo simulation model and launch

File: src/senton_description/urdf/senton.urdf.xacro (robot description, xacro)
@@ -18,4 +18,10 @@
         </material>
     </visual>
+    <collision>
+        <geometry>
+            <box size="${chassis_length} ${chassis_width} ${chassis_height}"/>
+        </geometry>
+        <origin xyz="0 0 ${chassis_z}" rpy="0 0 0"/>
+    </collision>
     <xacro:box_inertia
         m="${chassis_mass}"
@@ -46,4 +52,12 @@
             </material>
         </visual>
+        <collision>
+            <geometry>
+                <cylinder
+                    radius="${wheel_radius}"
+                    length="${wheel_width}"/>
+            </geometry>
+            <origin xyz="0 0 0" rpy="${pi/2} 0 0"/>
+        </collision>
         <xacro:cylinder_inertia
             m="${wheel_mass}"
@@ -56,5 +70,13 @@
 <!-- Front steering knuckle macro -->
 <xacro:macro name="steering_knuckle" params="name x y">
-    <link name="${name}_knuckle_link"/>
+    <link name="${name}_knuckle_link">
+    <xacro:box_inertia
+        m="${knuckle_mass}"
+        x="${knuckle_length}"
+        y="${knuckle_width}"
+        z="${knuckle_height}"
+        o_xyz="0 0 0"
+        o_rpy="0 0 0"/>
+</link>
     <joint name="${name}_steering_joint" type="revolute">
         <parent link="base_link"/>

File: src/senton_description/urdf/senton_properties.xacro (robot description, xacro)
@@ -17,5 +17,10 @@
     <xacro:property name="chassis_z"      value="0.03"/>
     <xacro:property name="chassis_mass"
-                value="${vehicle_mass - 4 * wheel_mass}"/>
+                value="${vehicle_mass - 4 * wheel_mass - 2 * knuckle_mass}"/>
+    <!-- Temporary steering knuckle approximation -->
+<xacro:property name="knuckle_mass" value="0.01"/>
+<xacro:property name="knuckle_length" value="0.02"/>
+<xacro:property name="knuckle_width" value="0.02"/>
+<xacro:property name="knuckle_height" value="0.02"/>
       <!-- Inertia macros -->
     <xacro:macro name="box_inertia" params="m x y z o_xyz o_rpy">

Commit message: Add ROS 2 control for steering and drive

File: src/senton_description/urdf/senton.urdf.xacro (robot description, xacro)
@@ -128,3 +128,44 @@
     y="${-track_width/2}"
 />
+<ros2_control name="GazeboSystem" type="system">
+    <hardware>
+        <plugin>gz_ros2_control/GazeboSimSystem</plugin>
+    </hardware>
+    <joint name="front_left_steering_joint" >
+        <command_interface name="position"/>
+        <state_interface name="position"/>
+        <state_interface  name="velocity"/>
+    </joint>
+    <joint name="front_right_steering_joint">
+        <command_interface name="position"/>
+        <state_interface name="position"/>
+        <state_interface name="velocity"/>
+    </joint>
+    <joint name="front_left_joint">
+        <command_interface name="velocity"/>
+        <state_interface name="position"/>
+        <state_interface name="velocity"/>
+    </joint>
+    <joint name="front_right_joint">
+        <command_interface name="velocity"/>
+        <state_interface name="position"/>
+        <state_interface name="velocity"/>
+    </joint>
+    <joint name="rear_left_joint">
+        <command_interface name="velocity"/>
+        <state_interface name="position"/>
+        <state_interface name="velocity"/>
+    </joint>
+    <joint name="rear_right_joint">
+        <command_interface name="velocity"/>
+        <state_interface name="position"/>
+        <state_interface name="velocity"/>
+    </joint>
+</ros2_control>
+<gazebo>
+    <plugin filename="gz_ros2_control-system"
+            name="gz_ros2_control::GazeboSimROS2ControlPlugin">
+        <parameters>$(find senton_description)/config/controllers.yaml</parameters>
+    </plugin>
+</gazebo>
 </robot>

Commit message: Add RPLIDAR simulation and ROS 2 scan bridge

File: src/senton_description/urdf/senton.urdf.xacro (robot description, xacro)
@@ -167,3 +167,58 @@
     </plugin>
 </gazebo>
+<link name="lidar_link">
+    <visual>
+        <geometry>
+            <cylinder radius="${lidar_radius}" length="${lidar_height}"/>
+        </geometry>
+        <material name="black">
+            <color rgba="0.05 0.05 0.05 1.0"/>
+        </material>
+    </visual>
+    <collision>
+        <geometry>
+            <cylinder radius="${lidar_radius}" length="${lidar_height}"/>
+        </geometry>
+    </collision>
+    <xacro:cylinder_inertia
+        m="${lidar_mass}"
+        r="${lidar_radius}"
+        l="${lidar_height}"
+        o_xyz="0 0 0"
+        o_rpy="0 0 0"/>
+</link>
+<joint name="lidar_joint" type="fixed">
+    <parent link="base_link"/>
+    <child link="lidar_link"/>
+    <origin xyz="0.16 0 0.13" rpy="0 0 0"/>
+</joint>
+<gazebo reference="lidar_link">
+    <sensor name="lidar_sensor" type="gpu_lidar">
+        <update_rate>10</update_rate>
+        <always_on>true</always_on>
+        <visualize>true</visualize>
+        <ray>
+            <scan>
+                <horizontal>
+                    <samples>3200</samples>
+                    <min_angle>-${pi}</min_angle>
+                    <max_angle>${pi}</max_angle>
+                </horizontal>
+                <vertical>
+                    <samples>1</samples>
+                    <resolution>1</resolution>
+                    <min_angle>0</min_angle>
+                    <max_angle>0</max_angle>
+                </vertical>
+            </scan>
+            <range>
+                <min>0.05</min>
+                <max>30.0</max>
+                <resolution>0.013</resolution>
+            </range>
+        </ray>
+        <topic>scan</topic>
+        <gz_frame_id>lidar_link</gz_frame_id>
+    </sensor>
+</gazebo>
 </robot>

File: src/senton_description/urdf/senton_properties.xacro (robot description, xacro)
@@ -1,32 +1,44 @@
 <?xml version="1.0"?>
 <robot xmlns:xacro="http://www.ros.org/wiki/xacro">
- <!-- vehicle dimensions-->
-     <xacro:property name="vehicle_length" value="0.558"/>
-     <xacro:property name="vehicle_width" value="0.305"/>
-     <xacro:property name="vehicle_height" value="0.210"/>
-     <xacro:property name="vehicle_mass" value="3.55"/>
-     <xacro:property name= "wheelbase" value="0.327"/>
-    <!-- wheel dimensions-->
-     <xacro:property name="wheel_radius" value="0.052"/>
-     <xacro:property name="wheel_width" value="0.042"/>
-     <xacro:property name="track_width" value="0.263"/>
-     <xacro:property name="wheel_mass" value="0.130"/>
-    <xacro:property name="chassis_length" value="0.40"/>
-    <xacro:property name="chassis_width"  value="0.16"/>
+    <!-- Vehicle dimensions -->
+    <xacro:property name="vehicle_length" value="0.558"/>
+    <xacro:property name="vehicle_width" value="0.305"/>
+    <xacro:property name="vehicle_height" value="0.210"/>
+    <xacro:property name="vehicle_mass" value="3.55"/>
+    <xacro:property name="wheelbase" value="0.327"/>
+    <!-- RPLIDAR S2-->
+    <xacro:property name="lidar_radius" value="0.0385"/>
+    <xacro:property name="lidar_height" value="0.03885"/>
+    <xacro:property name="lidar_mass" value = "0.190"/>
+    <!-- Wheel dimensions -->
+    <xacro:property name="wheel_radius" value="0.052"/>
+    <xacro:property name="wheel_width" value="0.042"/>
+    <xacro:property name="track_width" value="0.255"/>
+    <xacro:property name="wheel_mass" value="0.130"/>
+    <!-- Simplified chassis / tub dimensions -->
+    <xacro:property name="chassis_length" value="0.308"/>
+    <xacro:property name="chassis_width" value="0.157"/>
     <xacro:property name="chassis_height" value="0.09"/>
-    <xacro:property name="chassis_z"      value="0.03"/>
-    <xacro:property name="chassis_mass"
-                value="${vehicle_mass - 4 * wheel_mass - 2 * knuckle_mass}"/>
+    <xacro:property name="chassis_z" value="0.03"/>
     <!-- Temporary steering knuckle approximation -->
-<xacro:property name="knuckle_mass" value="0.01"/>
-<xacro:property name="knuckle_length" value="0.02"/>
-<xacro:property name="knuckle_width" value="0.02"/>
-<xacro:property name="knuckle_height" value="0.02"/>
-      <!-- Inertia macros -->
+    <xacro:property name="knuckle_mass" value="0.01"/>
+    <xacro:property name="knuckle_length" value="0.02"/>
+    <xacro:property name="knuckle_width" value="0.02"/>
+    <xacro:property name="knuckle_height" value="0.02"/>
+    <xacro:property
+        name="chassis_mass"
+        value="${vehicle_mass - 4 * wheel_mass - 2 * knuckle_mass}"/>
+    <!-- Inertia macros -->
     <xacro:macro name="box_inertia" params="m x y z o_xyz o_rpy">
         <inertial>
             <origin xyz="${o_xyz}" rpy="${o_rpy}"/>
             <mass value="${m}"/>
-            <inertia ixx="${(m / 12) * (y*y + z*z)}" ixy="0" ixz="0" iyy="${(m / 12) * (x*x + z*z)}" iyz="0" izz="${(m / 12) * (x*x + y*y)}"/>
+            <inertia
+                ixx="${(m / 12) * (y*y + z*z)}"
+                ixy="0"
+                ixz="0"
+                iyy="${(m / 12) * (x*x + z*z)}"
+                iyz="0"
+                izz="${(m / 12) * (x*x + y*y)}"/>
         </inertial>
     </xacro:macro>
@@ -35,5 +47,11 @@
             <origin xyz="${o_xyz}" rpy="${o_rpy}"/>
             <mass value="${m}"/>
-            <inertia ixx="${(m / 12) * (3*r*r + l*l)}" ixy="0" ixz="0" iyy="${(m / 12) * (3*r*r + l*l)}" iyz="0" izz="${(m / 2) * r*r}"/>
+            <inertia
+                ixx="${(m / 12) * (3*r*r + l*l)}"
+                ixy="0"
+                ixz="0"
+                iyy="${(m / 12) * (3*r*r + l*l)}"
+                iyz="0"
+                izz="${(m / 2) * r*r}"/>
         </inertial>
     </xacro:macro>
